File: imote1.brd (EAGLE design)
At the start: 17.8 x 43.2 mm, 20 parts, among them IC1 ATmega328P-AU, J3 USB-MINI-B%C, J4 HEAD3X2, Q1 16MHz

Commit message: ..
Parts:
- removed C2: 4.7uF, MySMD:TAN-A
- removed J4: HEAD3X2, MyCON2:HEAD3X2
- removed LED3: L_AMBER, MySMD:LED0805
- removed LED4: BLUE, MySMD:LED0805
- removed U$36: LOGO-G%117X105, MyBLK:LOGO-G_117X105
- removed U$37, U$4, U$53, U$54: FIDUCIAL1X2, SparkFun:FIDUCIAL-1X2
- added C1: 0.1uF, rcl:C2012
- added JP1: (no value), pinhead:2X03
- added LED1, LED2, TODO-IRLED1\: (no value), led:CHIP-LED0805
- added RB: 4.7k, resistor:R2012
- added RC: 47, resistor:R2012
- added T1: 2SC1815, transistor:TO92-ECB
- C3: value 0.1uF -> 10uF; device MySMD:CAP0805-NP -> rcl:E2,5-5
- moved C3 73.0 mm to (-18.1, -52.1), flipped to the top, turned to 0 degrees
Connections:
- new net D0/RX: IC1.30
- new net D1/TX: IC1.31
- new net D3/IRIN: IC1.1
- new net D9/IROUT: IC1.13, RB.2
- new net N$10: RB.1, T1.B
- new net N$11: RC.1, T1.C
- new net N$12: RC.2, TODO-IRLED1\.C
- new net N$4: IC1.17
- new net N$6: JP1.3
- new net N$8: JP1.5
- new net N$9: JP1.4
- net !RESET: no longer J4.5
- net +5V: now also C1.1, C3.+, JP1.2, TODO-IRLED1\.A; no longer C2.1, C3.1, J4.2
- net D11/MOSI: no longer J4.4
- net D12/MISO: now also JP1.1; no longer J4.1
- net D13/SCK: now also R2.2; no longer IC1.17, J4.3
- net GND: now also C1.2, C3.-, JP1.6, LED1.C, LED2.C, T1.E; no longer C2.2, C3.2, J4.6, LED3.1, LED4.1
- net N$1: now also Q1.1
- net N$2: now also Q1.2
- net N$3: now also LED1.A; no longer LED4.2
- net N$7: now also LED2.A, R2.1; no longer LED3.2
Routing:
- net +5V: track 95.7 -> 28.0 mm, vias 7 -> 1
- net D12/MISO: track 41.5 -> 0.00 mm
- net D11/MOSI: track 35.2 -> 0.00 mm
- net D13/SCK: track 27.6 -> 0.00 mm, vias 2 -> 0
- net !RESET: track 9.09 -> 0.00 mm
- net N$3: track 7.79 -> 0.00 mm, vias 1 -> 0
- net N$7: track 7.24 -> 0.00 mm, vias 1 -> 0
