File: iMote.brd (EAGLE design)
At the start: 17.8 x 43.2 mm, 19 parts, among them IC1 ATmega328P-AU, J3 USB-MINI-B%C, Q1 16MHz, T1 2SC1815

Commit message: ..
Parts:
- removed J3: USB-MINI-B%C, MyCON2:USB-MINI-B_2
- removed TODO-IRLED1\: (no value), led:CHIP-LED0805
- added C10: 1.0uF, rcl:C2012
- added C11: 0.01uF, rcl:C2012
- added C12: 4.7uF, rcl:C2012
- added C2, C7, C8, C9: 0.1uF, rcl:C2012
- added CN2: C-02235, akizukidenshi:C-02235
- added D1: IR, akizukidenshi:LED
- added IC2: BLE112-A-VISUAL, sf-bluegiga:BLE112-A
- added JP2: ICSP, pinhead:2X03
- added LED3: GREEN, led:CHIP-LED0805
- added LED4: RED, led:CHIP-LED0805
- added PL-IRM2161: PL-IRM2161, akizukidenshi:IR-RECEIVER
- added R4: 1K, resistor:R2012
- added R5, R6: 330, resistor:R2012
- added R7: 200, resistor:R2012
- added S2: B3F-1000, switch-omron:B3F-10XX
- added SJ1: 0, jumper:SJ
- added STANDOFF1, STANDOFF2, STANDOFF3, STANDOFF4: STAND-OFF, SparkFun-Electromechanical:STAND-OFF
- added U2: NJM2863, akizukidenshi:SOT23-5
- JP1: value (none) -> CC-HEADER; device pinhead:2X03 -> pinhead:2X05
- LED1: value (none) -> GREEN
- LED2: value (none) -> BLUE
- moved RC 182.6 mm to (58.2, 75.7)
- moved RB 180.0 mm to (73.5, 75.7)
- moved C3 149.8 mm to (69.7, 69.4)
- moved LED2 147.6 mm to (44.3, 74.5)
- moved LED1 147.1 mm to (49.4, 74.5)
- moved C1 134.5 mm to (63.3, 60.5)
- moved T1 133.8 mm to (28.1, 60.3)
- moved C6 125.8 mm to (57.0, 60.5)
- moved R2 116.2 mm to (68.4, 75.7)
- moved R3 115.8 mm to (63.3, 75.7)
- moved C4 114.0 mm to (50.6, 60.5)
- moved C5 113.6 mm to (44.3, 60.5)
- moved S1 107.6 mm to (71.0, 51.6)
- moved Q1 104.2 mm to (59.5, 50.3)
- moved R1 103.7 mm to (53.2, 75.7)
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Connections:
- removed net N$4: IC1.17
- removed net N$6: JP1.3
- removed net N$8: JP1.5
- removed net N$9: JP1.4
- new net !BLE/RST: IC2.RESET, JP1.7, R4.1, S2.1, S2.2
- new net +3V3: C10.1, C2.1, C7.1, C8.1, IC2.AVDD, IC2.AVDD@2, IC2.DVDD, IC2.VDD_USB, JP1.2, R4.2, R5.1, SJ1.2, U2.4
- new net BLE/P0_0: IC2.P0_0, R6.2
- new net BLE/P2_1: IC2.P2_1, JP1.4
- new net BLE/P2_2: IC2.P2_2, JP1.3
- new net N$13: LED4.A, R6.1
- new net N$14: C11.1, U2.3
- new net N$16: C12.1, PL-IRM2161.3, R7.1
- new net N$5: LED3.A, R5.2
- new net PRG/VDD: JP1.9, SJ1.1
- net !RESET: now also JP2.5
- net +5V: now also C9.1, CN2.VBUS, D1.A, JP2.2, R7.2, U2.1, U2.5; no longer J3.5, JP1.2, TODO-IRLED1\.A
- net D0/RX: now also IC2.P0_4
- net D1/TX: now also IC2.P0_5
- net D11/MOSI: now also JP2.4
- net D12/MISO: now also JP2.1; no longer JP1.1
- net D13/SCK: now also IC1.17, JP2.3
- net D3/IRIN: now also PL-IRM2161.1
- net GND: now also C10.2, C11.2, C12.2, C2.2, C7.2, C8.2, C9.2, CN2.GND, CN2.SH1, CN2.SH2, CN2.SH3, CN2.SH4, IC2.GND, IC2.GND@2, IC2.GND@3, IC2.GND@4, JP1.1, JP2.6, LED3.C, LED4.C, PL-IRM2161.2, S2.3, S2.4, U2.2; no longer J3.1, J3.6, J3.7, J3.8, J3.9, JP1.6
- net N$12: now also D1.C; no longer TODO-IRLED1\.C
Routing:
- net GND: track 4.36 -> 312.8 mm
- net +5V: track 28.0 -> 156.6 mm
- net N$2: track 0.00 -> 51.5 mm, vias 0 -> 2
- net N$10: track 0.00 -> 49.4 mm, vias 0 -> 1
- net N$11: track 0.00 -> 49.2 mm
- net N$12: track 0.00 -> 45.0 mm
- net !RESET: track 0.00 -> 36.5 mm, vias 0 -> 1
- net N$7: track 0.00 -> 24.8 mm, vias 0 -> 2
- net N$3: track 0.00 -> 18.1 mm, vias 0 -> 2
- net N$1: track 0.00 -> 13.5 mm
- removed copper zone on layer 1, net COM
- removed copper zone on layer 16, net COM
Other:
- board size 17.8 x 43.2 mm -> 100 x 80 mm
- board text removed: "*"
- board text removed: "1"
- board text removed: "2009"
- board text removed: "3V3"
- board text removed: "5V"
- board text removed: "A0"
- board text removed: "A1"
- board text removed: "A2"
- board text removed: "A3"
- board text removed: "A4"
- board text removed: "A5"
- board text removed: "A6"
- board text removed: "A7"
- board text removed: "ARDUINO"
- board text removed: "ARDUINO.CC"
- board text removed: "D10"
- board text removed: "D11"
- board text removed: "D12"
- board text removed: "D13"
- board text removed: "D2"
- board text removed: "D3"
- board text removed: "D4"
- board text removed: "D5"
- board text removed: "D6"
- board text removed: "D7"
- board text removed: "D8"
- board text removed: "D9"
- board text removed: "GND"
- board text removed: "GRAVITECH.US"
- board text removed: "ICSP"
- board text removed: "L"
- board text removed: "NANO"
- board text removed: "PWR"
- board text removed: "REF"
- board text removed: "RST"
- board text removed: "RX"
- board text removed: "RX0"
- board text removed: "TX"
- board text removed: "TX1"
- board text removed: "USA"
- board text removed: "V3.0"
- board text removed: "VIN"

Commit message: schematic complete?
Parts:
- removed C10: 1.0uF, rcl:C2012
- removed C11: 0.01uF, rcl:C2012
- removed C9: 0.1uF, rcl:C2012
- removed JP2: ICSP, pinhead:2X03
- removed U2: NJM2863, akizukidenshi:SOT23-5
- added C13, C14: 0.1uF, rcl:C2012
- added CN1: C-02235, akizukidenshi:C-02235
- added IC3: FT232RLSSOP, akizukidenshi:SSOP28DB
- added LED5: RED, led:CHIP-LED0805
- added LED6: GREEN, led:CHIP-LED0805
- added R8, R9: 680, resistor:R2012
- CN2: value C-02235 -> ICSP; device akizukidenshi:C-02235 -> pinhead:2X03
- moved CN2 30.0 mm to (70.0, 10.0), turned to 270 degrees
- renumbered JP1 to CN3
Connections:
- removed net D0/RX: IC1.30, IC2.P0_4
- removed net D1/TX: IC1.31, IC2.P0_5
- removed net D3/IRIN: IC1.1, PL-IRM2161.1
- removed net N$14: C11.1, U2.3
- new net D0/USBRX: IC1.30, IC3.1
- new net D1/USBTX: IC1.31, IC3.5
- new net D2/IRIN: IC1.32, PL-IRM2161.1
- new net D3/BLERX: IC1.1, IC2.P0_4
- new net D4/BLETX: IC1.2, IC2.P0_5
- new net N$4: LED5.A, R8.1
- new net N$6: LED6.A, R9.1
- new net N$8: C14.1, IC3.2
- new net USB/RXLED: IC3.22, R9.2
- new net USB/TXLED: IC3.23, R8.2
- new net USBD+: CN1.D+, IC3.15
- new net USBD-: CN1.D-, IC3.16
- net !RESET: now also C14.2, CN2.5; no longer JP2.5
- net +3V3: now also C13.1, IC3.17; no longer C10.1, U2.4
- net +5V: now also CN1.VBUS, CN2.2, IC3.20, IC3.4; no longer C9.1, CN2.VBUS, JP2.2, U2.1, U2.5
- net D11/MOSI: now also CN2.4; no longer JP2.4
- net D12/MISO: now also CN2.1; no longer JP2.1
- net D13/SCK: now also CN2.3; no longer JP2.3
- net GND: now also C13.2, CN1.GND, CN1.SH1, CN1.SH2, CN1.SH3, CN1.SH4, CN2.6, IC3.18, IC3.21, IC3.25, IC3.26, IC3.7, LED5.C, LED6.C; no longer C10.2, C11.2, C9.2, CN2.GND, CN2.SH1, CN2.SH2, CN2.SH3, CN2.SH4, JP2.6, U2.2

Commit message: irin/iroutをそれぞれD8,D3に移動
Connections:
- removed net D2/IRIN: IC1.32, PL-IRM2161.1
- removed net D3/BLERX: IC1.1, IC2.P0_4
- removed net D4/BLETX: IC1.2, IC2.P0_5
- removed net D9/IROUT: IC1.13, RB.2
- new net D3/IROUT: IC1.1, RB.2
- new net D4/BLERX: IC1.2, IC2.P0_4
- new net D5/BLETX: IC1.9, IC2.P0_5
- new net D8/IRIN: IC1.12, PL-IRM2161.1
Changed lines of the file:
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@@
 <wire x1="62.23" y1="33.02" x2="-18.73" y2="-180" width="0" layer="19" extent="1-1"/>
-</signal>
-<signal name="D9/IROUT">
-<contactref element="IC1" pad="13"/>
-<contactref element="RB" pad="2"/>
-<wire x1="32.3" y1="40.7874" x2="74.34" y2="75.72" width="0" layer="19" extent="1-1"/>
 </signal>
 <signal name="+3V3">
@@
 <wire x1="2.54" y1="-160" x2="-0.85" y2="-170" width="0" layer="19" extent="1-1"/>
 </signal>
-<signal name="D2/IRIN">
-<contactref element="IC1" pad="32"/>
-<contactref element="PL-IRM2161" pad="1"/>
-<wire x1="29.1" y1="49.3726" x2="-2.54" y2="-160" width="0" layer="19" extent="1-1"/>
-</signal>
-<signal name="D3/BLERX">
-<contactref element="IC1" pad="1"/>
-<contactref element="IC2" pad="P0_4"/>
-<wire x1="16" y1="45.65" x2="27.6074" y2="47.88" width="0" layer="19" extent="1-1"/>
-</signal>
-<signal name="D4/BLETX">
-<contactref element="IC1" pad="2"/>
-<contactref element="IC2" pad="P0_5"/>
-<wire x1="16" y1="44.4" x2="27.6074" y2="47.08" width="0" layer="19" extent="1-1"/>
-</signal>
 <signal name="D0/USBRX">
 <contactref element="IC1" pad="30"/>
@@
 <wire x1="-10" y1="-231.05" x2="-20.85" y2="-230" width="0" layer="19" extent="1-1"/>
 </signal>
+<signal name="D8/IRIN">
+<contactref element="IC1" pad="12"/>
+<contactref element="PL-IRM2161" pad="1"/>
+<wire x1="31.5" y1="40.7874" x2="-2.54" y2="-160" width="0" layer="19" extent="1-1"/>
+</signal>
+<signal name="D3/IROUT">
+<contactref element="IC1" pad="1"/>
+<contactref element="RB" pad="2"/>
+<wire x1="27.6074" y1="47.88" x2="74.34" y2="75.72" width="0" layer="19" extent="1-1"/>
+</signal>
+<signal name="D4/BLERX">
+<contactref element="IC1" pad="2"/>
+<contactref element="IC2" pad="P0_4"/>
+<wire x1="16" y1="45.65" x2="27.6074" y2="47.08" width="0" layer="19" extent="1-1"/>
+</signal>
+<signal name="D5/BLETX">
+<contactref element="IC1" pad="9"/>
+<contactref element="IC2" pad="P0_5"/>
+<wire x1="16" y1="44.4" x2="29.1" y2="40.7874" width="0" layer="19" extent="1-1"/>
+</signal>
 </signals>

Commit message: TLN105B(F)の抵抗値入れた
Parts:
- D1: value IR -> TLN105B(F)
- RB: value 4.7k -> 470
- RC: value 47 -> 4.7
Changed lines of the file:
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@@
 <element name="LED2" library="led" package="CHIP-LED0805" value="BLUE" x="44.28" y="74.45"/>
 <element name="T1" library="transistor" package="TO92-ECB" value="2SC1815" x="28.09" y="60.32"/>
-<element name="RB" library="resistor" package="R2012" value="4.7k" x="73.49" y="75.72"/>
-<element name="RC" library="resistor" package="R2012" value="47" x="58.25" y="75.72"/>
+<element name="RB" library="resistor" package="R2012" value="470" x="73.49" y="75.72"/>
+<element name="RC" library="resistor" package="R2012" value="4.7" x="58.25" y="75.72"/>
 <element name="STANDOFF1" library="SparkFun-Electromechanical" package="STAND-OFF" value="STAND-OFF" x="93.33" y="9.37"/>
 <element name="STANDOFF2" library="SparkFun-Electromechanical" package="STAND-OFF" value="STAND-OFF" x="6.98" y="9.37"/>
@@
 <element name="R7" library="resistor" package="R2012" value="200" x="0" y="-170"/>
 <element name="C12" library="rcl" package="C2012" value="4.7uF" x="0" y="-180"/>
-<element name="D1" library="akizukidenshi" package="LED" value="IR" x="-20" y="-180"/>
+<element name="D1" library="akizukidenshi" package="LED" value="TLN105B(F)" x="-20" y="-180"/>
 <element name="IC3" library="akizukidenshi" package="SSOP28DB" value="FT232RLSSOP" x="-10" y="-190">
 <attribute name="PROD_ID" value="IC-00870" x="-10" y="-190" size="1.778" layer="27" display="off"/>

Commit message: 基板設計中
Parts:
- removed STANDOFF3: STAND-OFF, SparkFun-Electromechanical:STAND-OFF
- moved C13 234.1 mm to (7.94, 32.4)
- moved C14 234.1 mm to (7.94, 22.4)
- moved LED5 234.1 mm to (17.9, 12.4)
- moved LED6 234.1 mm to (17.9, 2.41)
- moved R8 234.1 mm to (7.94, 12.4)
- moved R9 234.1 mm to (7.94, 2.41)
- moved IC3 232.4 mm to (53.5, 33.5)
- moved D1 205.0 mm to (37.1, 16.9)
- moved C12 183.4 mm to (25.4, 1.61)
- moved PL-IRM2161 183.4 mm to (25.4, 21.6)
- moved R7 183.4 mm to (25.4, 11.6)
- moved SJ1 183.4 mm to (25.4, 31.6)
- moved CN3 163.6 mm to (76.2, 4.78)
- moved LED4 134.6 mm to (84.9, 21.8)
- moved R6 134.6 mm to (84.9, 31.8)
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Routing:
- net GND: track 312.8 -> 0.02 mm
- net +5V: track 156.6 -> 0.00 mm, vias 1 -> 0
- net N$2: track 51.5 -> 0.00 mm, vias 2 -> 0
- net N$10: track 49.4 -> 0.00 mm, vias 1 -> 0
- net N$11: track 49.2 -> 0.00 mm
- net N$12: track 45.0 -> 0.00 mm
- net !RESET: track 36.5 -> 0.00 mm, vias 1 -> 0
- net N$7: track 24.8 -> 0.00 mm, vias 2 -> 0
- net N$3: track 18.1 -> 0.00 mm, vias 2 -> 0
- net N$1: track 13.5 -> 0.00 mm
- net +3V3: track 0.00 -> 1.83 mm

Commit message: ir led changed to OSIR5113A
Parts:
- D1: value TLN105B(F) -> OSIR5113A
- RB: value 470 -> 4.7k
- RC: value 4.7 -> 47
Changed lines of the file:
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@@
 <element name="LED2" library="led" package="CHIP-LED0805" value="BLUE" x="44.28" y="74.45"/>
 <element name="T1" library="transistor" package="TO92-ECB" value="2SC1815" x="28.09" y="60.32"/>
-<element name="RB" library="resistor" package="R2012" value="470" x="73.49" y="75.72"/>
-<element name="RC" library="resistor" package="R2012" value="4.7" x="58.25" y="75.72"/>
+<element name="RB" library="resistor" package="R2012" value="4.7k" x="73.49" y="75.72"/>
+<element name="RC" library="resistor" package="R2012" value="47" x="58.25" y="75.72"/>
 <element name="STANDOFF1" library="SparkFun-Electromechanical" package="STAND-OFF" value="STAND-OFF" x="95.87" y="4.29"/>
 <element name="STANDOFF2" library="SparkFun-Electromechanical" package="STAND-OFF" value="STAND-OFF" x="3.678" y="4.208"/>
@@
 <element name="R7" library="resistor" package="R2012" value="200" x="25.4" y="11.61"/>
 <element name="C12" library="rcl" package="C2012" value="4.7uF" x="25.4" y="1.61"/>
-<element name="D1" library="akizukidenshi" package="LED" value="TLN105B(F)" x="37.15" y="16.85"/>
+<element name="D1" library="akizukidenshi" package="LED" value="OSIR5113A" x="37.15" y="16.85"/>
 <element name="IC3" library="akizukidenshi" package="SSOP28DB" value="FT232RLSSOP" x="53.5" y="33.52">
 <attribute name="PROD_ID" value="IC-00870" x="53.5" y="33.52" size="1.778" layer="27" display="off"/>

Commit message: routing..
Parts:
- removed C12: 4.7uF, rcl:C2012
- removed C13, C14: 0.1uF, rcl:C2012
- removed PL-IRM2161: PL-IRM2161, akizukidenshi:IR-RECEIVER
- added C10: 4.7uF, rcl:C2012
- added C9: 0.1uF, rcl:C2012
- added PL-IRM1: PL-IRM2161, akizukidenshi:IR-RECEIVER
- C1, C2: value 0.1uF -> 22pF
- C3: value 10uF -> 0.1uF; device rcl:E2,5-5 -> rcl:C2012
- C4, C5: value 22pF -> 0.1uF
- C8: value 0.1uF -> 10uF; device rcl:C2012 -> rcl:E2,5-5
- IC2: value BLE112-A-VISUAL -> FT232RLSSOP; device sf-bluegiga:BLE112-A -> akizukidenshi:SSOP28DB
- IC3: value FT232RLSSOP -> BLE112-A-VISUAL; device akizukidenshi:SSOP28DB -> sf-bluegiga:BLE112-A
- LED1: value GREEN -> 5V
- LED2: value BLUE -> ICSP
- LED3: value GREEN -> 3.3V
- LED4: value RED -> BLE
- LED5: value RED -> USB/TX
- LED6: value GREEN -> USB/RX
- R7: value 200 -> 680
- R9: value 680 -> 200
- moved CN1 104.5 mm to (11.6, 75.6), turned to 180 degrees
- moved CN3 74.6 mm to (91.4, 77.8), turned to 180 degrees
- moved LED6 73.9 mm to (24.3, 76.1)
- moved IC2 72.2 mm to (19.8, 58.6), turned to 90 degrees
- moved RB 71.7 mm to (17.0, 31.6), turned to 90 degrees
- moved RC 68.3 mm to (19.8, 19.2), turned to 270 degrees
- moved CN2 64.8 mm to (30.6, 35.4)
- moved LED5 63.5 mm to (19.2, 75.9)
- moved R3 63.5 mm to (29.4, 22.1), turned to 180 degrees
- moved C8 63.3 mm to (8.41, 67.5), turned to 270 degrees
- moved C1 62.8 mm to (2.37, 45.2)
- moved R8 60.6 mm to (24.0, 70.8), turned to 270 degrees
- moved R7 59.6 mm to (18.8, 70.8), turned to 270 degrees
- moved C7 58.8 mm to (3.64, 68.1), turned to 270 degrees
- moved LED3 58.2 mm to (37.9, 76.0)
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- renumbered STANDOFF4 to STANDOFF3
Connections:
- net !BLE/RST: now also IC3.RESET; no longer IC2.RESET
- net !RESET: now also C5.2; no longer C14.2
- net +3V3: now also C4.1, C6.1, C9.1, IC2.17, IC3.AVDD, IC3.AVDD@2, IC3.DVDD, IC3.VDD_USB; no longer C13.1, C2.1, C7.1, C8.1, IC2.AVDD, IC2.AVDD@2, IC2.DVDD, IC2.VDD_USB, IC3.17
- net +5V: now also C7.1, C8.+, IC2.20, IC2.4, R2.1, R9.2; no longer C1.1, C3.+, IC3.20, IC3.4, R3.1, R7.2
- net AREF: now also C3.2; no longer C6.2
- net BLE/P0_0: now also IC3.P0_0; no longer IC2.P0_0
- net BLE/P2_1: now also IC3.P2_1; no longer IC2.P2_1
- net BLE/P2_2: now also IC3.P2_2; no longer IC2.P2_2
- net D0/USBRX: now also IC2.1; no longer IC3.1
- net D1/USBTX: now also IC2.5; no longer IC3.5
- net D13/SCK: now also R3.2; no longer R2.2
- net D4/BLERX: now also IC3.P0_4; no longer IC2.P0_4
- net D5/BLETX: now also IC3.P0_5; no longer IC2.P0_5
- net D8/IRIN: now also PL-IRM1.1; no longer PL-IRM2161.1
- net GND: now also C1.1, C10.2, C2.1, C3.1, C4.2, C6.2, C8.-, C9.2, IC2.18, IC2.21, IC2.25, IC2.26, IC2.7, IC3.GND, IC3.GND@2, IC3.GND@3, IC3.GND@4, PL-IRM1.2; no longer C1.2, C12.2, C13.2, C2.2, C3.-, C4.1, C5.1, C6.1, C8.2, IC2.GND, IC2.GND@2, IC2.GND@3, IC2.GND@4, IC3.18, IC3.21, IC3.25, IC3.26, IC3.7, PL-IRM2161.2
- net N$1: now also C2.2; no longer C4.2
- net N$16: now also C10.1, PL-IRM1.3, R9.1; no longer C12.1, PL-IRM2161.3, R7.1
- net N$2: now also C1.2; no longer C5.2
- net N$3: now also R2.2; no longer R3.2
- net N$4: now also R7.1; no longer R8.1
- net N$6: now also R8.1; no longer R9.1
- net N$7: now also R3.1; no longer R2.1
- net N$8: now also C5.1, IC2.2; no longer C14.1, IC3.2
- net USB/RXLED: now also IC2.22, R8.2; no longer IC3.22, R9.2
- net USB/TXLED: now also IC2.23, R7.2; no longer IC3.23, R8.2
- net USBD+: now also IC2.15; no longer IC3.15
- net USBD-: now also IC2.16; no longer IC3.16
Routing:
- net +3V3: track 1.83 -> 0.00 mm

Commit message: added git-revision
Parts:
- added U$1: 4fdebe4, git-revision:GIT-REVISION
Changed lines of the file:
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@@
 <element name="R8" library="resistor" package="R2012" value="680" x="24" y="70.8" rot="R270"/>
 <element name="LED6" library="led" package="CHIP-LED0805" value="USB/RX" x="24.29" y="76.07"/>
+<element name="U$1" library="git-revision" package="GIT-REVISION" value="4fdebe4" x="1.27" y="-2.54"/>
 </elements>
 <signals>
